File: universalModule/hardware/controlBoard/controlBoard.kicad_pcb (KiCad board)
At the start: 2 copper layers, 245.9 x 74 mm, 173 parts, among them J1 ESP_JTAG, J10 BATT_1, J11 BATT_3, J12 BATT_2, J13 PWR_1, J14 BATT_2, J15 PWR_3, J16 CTL_3, J17 CTL_1, J18 CTL_2, J19 PWR_4, J2 OLED_DISPLAY, J20 CTL_5, J21 CTL_4, J22 INT_1, J3 USB_ALT, J4 ShoeAConnectors, J5 MOTOR_BUS, J6 MOTOR_BUS_ALT, J7 ShoeBConnectors, J8 BIOS_SWD, J9 USB_C_Receptacle_USB2.0, Q1 SiA449DJ, Q2 SiA449DJ, Q3 SSM3K72CFS, Q4 BC817, Q5 BC817, SW1 SW_Push, SW2 STOP_BUTTON, SW3 SW_Push, SW4 START_BUTTON, SW5 SW_Push, U1 MP3431, U2 MP3431, U3 MP1496, U4 MP2615, U5 BQ29200, U6 ESP32-WROVER, U7 ICM-20948, U8 CP2102N-A01-GQFN28, U9 STM32F030C8Tx

Commit message: universalModule: Fine tune the control board
Parts:
- added H1: MountingHole, MountingHole:MountingHole_2.1mm, F.Cu at (271.5, 134.8)
- added H2: MountingHole, MountingHole:MountingHole_2.1mm, F.Cu at (216.5, 95.0)
- added H3: MountingHole, MountingHole:MountingHole_2.1mm, F.Cu at (271.5, 105.2)
- added H4: MountingHole, MountingHole:MountingHole_2.1mm, F.Cu at (216.5, 145.0)
- added H5: MountingHole, MountingHole:MountingHole_2.1mm, F.Cu at (39.0, 140.0)
- added H6: MountingHole, MountingHole:MountingHole_2.1mm, F.Cu at (39.0, 100.0)
- moved SW4 0.30 mm to (47.0, 103.5)
Other:
- outline, holes or cut-outs redrawn
- board text added: "3V3"
- board text added: "BATT"
- board text added: "E3 E2 E1 DA G VD IN EX CK G"
- board text added: "GND VDD MRX MTX INT EXT SCK DAT CE4 CE5 CE6 GND"
- board text added: "GND VDD RX TX"
- board text added: "INT"
- board text added: "IO 3V G CL RS G"
- board text added: "RX TX SDA SCL"
- board text added: "RoFI Universal Module - Battery Board v0.1 11/2019"
- board text added: "RoFI Universal Module - Control Board v0.1 11/2019"
- board text added: "RoFI Universal Module - Power Board v0.1 11/2019"
- board text added: "RoFI Universal Module UI Board v0.1 11/2019"
- board text added: "TMS TCK TDO TDI"
- board text added: "USB"
