File: hardwareModules/RoFICoM/hardware/control_board/bi-switch.sch (KiCad schematic (older format))
At the start: 11 parts, among them Q1 DMP6050SFG, Q2 SSM3K72CFS, Q3 DMP6050SFG, U6 ACS70331

Commit message: universalModule: Prepare electronics v0.2
Parts:
- removed Q3: DMP6050SFG, rofi:POWERDI_3333-8, symbol Device:Q_PMOS_GSD
- added Q3: AONR21357, rofi:DFN3.3X3.3-EP, symbol Device:Q_PMOS_SGD
- C6: value 470n -> 1u; LCSC (none) -> C52923
- D2: value 15V BZT52C15T-7 -> 15V EDZVT2R15B; JLCPCB_CORRECTION (none) -> 0;0;180; LCSC (none) -> C209631
- Q1: value DMP6050SFG -> AONR21357; footprint rofi:POWERDI_3333-8 -> rofi:DFN3.3X3.3-EP; symbol Device:Q_PMOS_GSD -> Device:Q_PMOS_SGD; JLCPCB_CORRECTION (none) -> 0;0;-90; LCSC (none) -> C431196
- Q2: value SSM3K72CFS -> PNM723T703E0-2; footprint Package_TO_SOT_SMD:SOT-416 -> Package_TO_SOT_SMD:SOT-723; JLCPCB_CORRECTION (none) -> 0;0;180; LCSC (none) -> C110713; manf# SSM3K72CFS,LF -> (none)
- R2: LCSC (none) -> C25917
- R3, R4, R5, R6: LCSC (none) -> C25741
- U6: JLCPCB_IGNORE (none) -> YES
Connections:
- net at D2.2 (A), R4.2, R6.1: now also Q1.2 (G), Q3.2 (G); no longer Q1.1 (G)
- net at D2.1 (K), R4.1: now also Q1.1 (S), Q3.1 (S); no longer Q1.2 (S)
- net at R3.2, U6.3 (IP-): now also Q3.3 (D)
Changed lines of the file:
@@
 $Descr A4 11693 8268
 encoding utf-8
-Sheet 3 3
+Sheet 2 4
 Title ""
 Date ""
@@
 $EndDescr
 $Comp
-L Device:Q_PMOS_GSD Q?
-U 1 1 5C87EAB3
-P 5750 3100
-AR Path="/5C87EAB3" Ref="Q?"  Part="1"
-AR Path="/5C87E670/5C87EAB3" Ref="Q3"  Part="1"
-AR Path="/5C883562/5C87EAB3" Ref="Q6"  Part="1"
-F 0 "Q6" V 6093 3100 50  0000 C CNN
-F 1 "DMP6050SFG" V 6002 3100 50  0000 C CNN
-F 2 "rofi:POWERDI_3333-8" H 5950 3200 50  0001 C CNN
-F 3 "~" H 5750 3100 50  0001 C CNN
-	1    5750 3100
-	0    1    -1   0
-$EndComp
-$Comp
 L rofi:ACS70331 U?
 U 1 1 5C87EABA
@@
 AR Path="/5C87E670/5C87EABA" Ref="U6"  Part="1"
 AR Path="/5C883562/5C87EABA" Ref="U7"  Part="1"
-F 0 "U7" H 6750 3200 50  0000 L CNN
+F 0 "U6" H 6750 3200 50  0000 L CNN
 F 1 "ACS70331" H 6300 3200 50  0000 L CNN
 F 2 "rofi:ACS70331" H 6400 2800 50  0001 C CNN
 F 3 "" H 6400 2800 50  0001 C CNN
+F 4 "YES" H 6600 3000 50  0001 C CNN "JLCPCB_IGNORE"
 	1    6600 3000
 	1    0    0    -1
 $EndComp
 $Comp
-L Device:Q_PMOS_GSD Q?
+L Device:Q_PMOS_SGD Q?
 U 1 1 5C87EAC1
 P 4250 3100
@@
 AR Path="/5C87E670/5C87EAC1" Ref="Q1"  Part="1"
 AR Path="/5C883562/5C87EAC1" Ref="Q4"  Part="1"
-F 0 "Q4" V 4593 3100 50  0000 C CNN
-F 1 "DMP6050SFG" V 4502 3100 50  0000 C CNN
-F 2 "rofi:POWERDI_3333-8" H 4450 3200 50  0001 C CNN
+F 0 "Q1" V 4593 3100 50  0000 C CNN
+F 1 "AONR21357" V 4502 3100 50  0000 C CNN
+F 2 "rofi:DFN3.3X3.3-EP" H 4450 3200 50  0001 C CNN
 F 3 "~" H 4250 3100 50  0001 C CNN
+F 4 "C431196" V 4250 3100 50  0001 C CNN "LCSC"
+F 5 "0;0;-90" V 4250 3100 50  0001 C CNN "JLCPCB_CORRECTION"
 	1    4250 3100
 	0    -1   -1   0
@@
 AR Path="/5C87E670/5C87EACB" Ref="D2"  Part="1"
 AR Path="/5C883562/5C87EACB" Ref="D3"  Part="1"
-F 0 "D3" V 4804 3229 50  0000 L CNN
-F 1 "15V BZT52C15T-7" V 4895 3229 50  0000 L CNN
+F 0 "D2" V 4804 3229 50  0000 L CNN
+F 1 "15V EDZVT2R15B" V 4895 3229 50  0000 L CNN
 F 2 "Diode_SMD:D_SOD-523" H 4850 3150 50  0001 C CNN
 F 3 "~" H 4850 3150 50  0001 C CNN
+F 4 "C209631" V 4850 3150 50  0001 C CNN "LCSC"
+F 5 "0;0;180" V 4850 3150 50  0001 C CNN "JLCPCB_CORRECTION"
 	1    4850 3150
 	0    1    1    0
@@
 AR Path="/5C87E670/5C87EAD3" Ref="R4"  Part="1"
 AR Path="/5C883562/5C87EAD3" Ref="R9"  Part="1"
-F 0 "R9" H 4570 3196 50  0000 L CNN
+F 0 "R4" H 4570 3196 50  0000 L CNN
 F 1 "100k" H 4570 3105 50  0000 L CNN
 F 2 "Resistor_SMD:R_0402_1005Metric" V 4430 3150 50  0001 C CNN
 F 3 "~" H 4500 3150 50  0001 C CNN
+F 4 "C25741" H 4500 3150 50  0001 C CNN "LCSC"
 	1    4500 3150
 	1    0    0    -1
@@
 AR Path="/5C87E670/5C87EAE6" Ref="R6"  Part="1"
 AR Path="/5C883562/5C87EAE6" Ref="R11"  Part="1"
-F 0 "R11" H 4920 3596 50  0000 L CNN
+F 0 "R6" H 4920 3596 50  0000 L CNN
 F 1 "100k" H 4920 3505 50  0000 L CNN
 F 2 "Resistor_SMD:R_0402_1005Metric" V 4780 3550 50  0001 C CNN
 F 3 "~" H 4850 3550 50  0001 C CNN
+F 4 "C25741" H 4850 3550 50  0001 C CNN "LCSC"
 	1    4850 3550
-	1    0    0    -1
-$EndComp
-$Comp
-L Device:Q_NMOS_GSD Q?
-U 1 1 5C87EAED
-P 4750 3900
-AR Path="/5C87EAED" Ref="Q?"  Part="1"
-AR Path="/5C87E670/5C87EAED" Ref="Q2"  Part="1"
-AR Path="/5C883562/5C87EAED" Ref="Q5"  Part="1"
-F 0 "Q5" H 4956 3946 50  0000 L CNN
-F 1 "SSM3K72CFS" H 4956 3855 50  0000 L CNN
-F 2 "Package_TO_SOT_SMD:SOT-416" H 4950 4000 50  0001 C CNN
-F 3 "~" H 4750 3900 50  0001 C CNN
-F 4 "SSM3K72CFS,LF" H 4750 3900 50  0001 C CNN "manf#"
-	1    4750 3900
 	1    0    0    -1
 $EndComp
@@
 AR Path="/5C87E670/5C87EAF4" Ref="R5"  Part="1"
 AR Path="/5C883562/5C87EAF4" Ref="R10"  Part="1"
-F 0 "R10" V 4293 4150 50  0000 C CNN
+F 0 "R5" V 4293 4150 50  0000 C CNN
 F 1 "100k" V 4384 4150 50  0000 C CNN
 F 2 "Resistor_SMD:R_0402_1005Metric" V 4430 4150 50  0001 C CNN
 F 3 "~" H 4500 4150 50  0001 C CNN
+F 4 "C25741" V 4500 4150 50  0001 C CNN "LCSC"
 	1    4500 4150
 	0    1    1    0
@@
 AR Path="/5C87E670/5C87EB01" Ref="#PWR0130"  Part="1"
 AR Path="/5C883562/5C87EB01" Ref="#PWR0136"  Part="1"
-F 0 "#PWR0136" H 4850 4050 50  0001 C CNN
+F 0 "#PWR0130" H 4850 4050 50  0001 C CNN
 F 1 "GND" H 4855 4127 50  0000 C CNN
 F 2 "" H 4850 4300 50  0001 C CNN
@@
 AR Path="/5C87E670/5C87ED9B" Ref="R3"  Part="1"
 AR Path="/5C883562/5C87ED9B" Ref="R8"  Part="1"
-F 0 "R8" H 6070 2496 50  0000 L CNN
+F 0 "R3" H 6070 2496 50  0000 L CNN
 F 1 "100k" H 6070 2405 50  0000 L CNN
 F 2 "Resistor_SMD:R_0402_1005Metric" V 5930 2450 50  0001 C CNN
 F 3 "~" H 6000 2450 50  0001 C CNN
+F 4 "C25741" H 6000 2450 50  0001 C CNN "LCSC"
 	1    6000 2450
 	1    0    0    -1
@@
 AR Path="/5C87E670/5C87F018" Ref="R2"  Part="1"
 AR Path="/5C883562/5C87F018" Ref="R7"  Part="1"
-F 0 "R7" H 6070 2196 50  0000 L CNN
+F 0 "R2" H 6070 2196 50  0000 L CNN
 F 1 "6k8" H 6070 2105 50  0000 L CNN
 F 2 "Resistor_SMD:R_0402_1005Metric" V 5930 2150 50  0001 C CNN
 F 3 "~" H 6000 2150 50  0001 C CNN
+F 4 "C25917" H 6000 2150 50  0001 C CNN "LCSC"
 	1    6000 2150
 	1    0    0    -1
@@
 AR Path="/5C87E670/5C87F066" Ref="#PWR0131"  Part="1"
 AR Path="/5C883562/5C87F066" Ref="#PWR0137"  Part="1"
-F 0 "#PWR0137" H 6000 1750 50  0001 C CNN
+F 0 "#PWR0131" H 6000 1750 50  0001 C CNN
 F 1 "GND" H 6005 1827 50  0000 C CNN
 F 2 "" H 6000 2000 50  0001 C CNN
@@
 AR Path="/5C87E670/5C87F338" Ref="#PWR0132"  Part="1"
 AR Path="/5C883562/5C87F338" Ref="#PWR0138"  Part="1"
-F 0 "#PWR0138" H 7050 2850 50  0001 C CNN
+F 0 "#PWR0132" H 7050 2850 50  0001 C CNN
 F 1 "GND" H 7055 2927 50  0000 C CNN
 F 2 "" H 7050 3100 50  0001 C CNN
@@
 AR Path="/5C87E670/5C87FC70" Ref="#PWR0133"  Part="1"
 AR Path="/5C883562/5C87FC70" Ref="#PWR0139"  Part="1"
-F 0 "#PWR0139" H 6800 3250 50  0001 C CNN
+F 0 "#PWR0133" H 6800 3250 50  0001 C CNN
 F 1 "GND" H 6805 3327 50  0000 C CNN
 F 2 "" H 6800 3500 50  0001 C CNN
@@
 AR Path="/5C87E670/5C87FCE8" Ref="#PWR0134"  Part="1"
 AR Path="/5C883562/5C87FCE8" Ref="#PWR0140"  Part="1"
-F 0 "#PWR0140" H 7500 2750 50  0001 C CNN
+F 0 "#PWR0134" H 7500 2750 50  0001 C CNN
 F 1 "+3V3" V 7515 3028 50  0000 L CNN
 F 2 "" H 7500 2900 50  0001 C CNN
@@
 AR Path="/5C87E670/5C8800BB" Ref="C6"  Part="1"
 AR Path="/5C883562/5C8800BB" Ref="C7"  Part="1"
-F 0 "C7" H 7315 2796 50  0000 L CNN
-F 1 "470n" H 7315 2705 50  0000 L CNN
+F 0 "C6" H 7315 2796 50  0000 L CNN
+F 1 "1u" H 7315 2705 50  0000 L CNN
 F 2 "Capacitor_SMD:C_0402_1005Metric" H 7238 2600 50  0001 C CNN
 F 3 "~" H 7200 2750 50  0001 C CNN
+F 4 "C52923" H 7200 2750 50  0001 C CNN "LCSC"
 	1    7200 2750
 	1    0    0    -1
@@
 AR Path="/5C87E670/5C88011B" Ref="#PWR0135"  Part="1"
 AR Path="/5C883562/5C88011B" Ref="#PWR0141"  Part="1"
-F 0 "#PWR0141" H 7200 2350 50  0001 C CNN
+F 0 "#PWR0135" H 7200 2350 50  0001 C CNN
 F 1 "GND" H 7205 2427 50  0000 C CNN
 F 2 "" H 7200 2600 50  0001 C CNN
@@
 Wire Wire Line
 	6150 2650 6150 2900
+$Comp
+L Device:Q_PMOS_SGD Q?
+U 1 1 60E738F0
+P 5750 3100
+AR Path="/60E738F0" Ref="Q?"  Part="1"
+AR Path="/5C87E670/60E738F0" Ref="Q3"  Part="1"
+AR Path="/5C883562/60E738F0" Ref="Q6"  Part="1"
+F 0 "Q3" V 6093 3100 50  0000 C CNN
+F 1 "AONR21357" V 6002 3100 50  0000 C CNN
+F 2 "rofi:DFN3.3X3.3-EP" H 5950 3200 50  0001 C CNN
+F 3 "~" H 5750 3100 50  0001 C CNN
+F 4 "C431196" V 5750 3100 50  0001 C CNN "LCSC"
+F 5 "0;0;-90" V 5750 3100 50  0001 C CNN "JLCPCB_CORRECTION"
+	1    5750 3100
+	0    1    -1   0
+$EndComp
+$Comp
+L Device:Q_NMOS_GSD Q2
+U 1 1 60E77B8E
+P 4750 3900
+AR Path="/5C87E670/60E77B8E" Ref="Q2"  Part="1"
+AR Path="/5C883562/60E77B8E" Ref="Q5"  Part="1"
+F 0 "Q2" H 4954 3946 50  0000 L CNN
+F 1 "PNM723T703E0-2" H 4954 3855 50  0000 L CNN
+F 2 "Package_TO_SOT_SMD:SOT-723" H 4950 4000 50  0001 C CNN
+F 3 "~" H 4750 3900 50  0001 C CNN
+F 4 "C110713" H 4750 3900 50  0001 C CNN "LCSC"
+F 5 "0;0;180" H 4750 3900 50  0001 C CNN "JLCPCB_CORRECTION"
+	1    4750 3900
+	1    0    0    -1
+$EndComp
 $EndSCHEMATC
