File: hardwareModules/universalModule/hardware/controlBoard/controlBoard.kicad_pcb (KiCad board)
At the start: 2 copper layers, 245.9 x 74 mm, 179 parts, among them J1 ESP_JTAG, J10 BATT_1, J11 BATT_3, J12 BATT_2, J13 PWR_1, J14 BATT_2, J15 PWR_3, J16 CTL_3, J17 CTL_1, J18 CTL_2, J19 PWR_4, J2 OLED_DISPLAY, J20 CTL_5, J21 CTL_4, J22 INT_1, J3 USB_ALT, J4 ShoeAConnectors, J5 MOTOR_BUS, J6 MOTOR_BUS_ALT, J7 ShoeBConnectors, J8 BIOS_SWD, J9 USB_C_Receptacle_USB2.0, Q1 SiA449DJ, Q2 SiA449DJ, Q3 SSM3K72CFS, Q4 BC817, Q5 BC817, SW1 SW_Push, SW2 STOP_BUTTON, SW3 SW_Push, SW4 START_BUTTON, SW5 SW_Push, U1 MP3431, U2 MP3431, U3 MP1496, U4 MP2615, U5 BQ29200, U6 ESP32-WROVER, U7 ICM-20948, U8 CP2102N-A01-GQFN28, U9 STM32F030C8Tx

Commit message: universalModule: Draft schematics of the new version of the control board
Parts:
- removed D10: YELLOW, LED_SMD:LED_0603_1608Metric
- removed D15: GREEN, LED_SMD:LED_0603_1608Metric
- removed D5: PMEG045V100EPDAZ, rofi:D_SOT1289
- removed D6, D7: BAT54J,115, Diode_SMD:D_SOD-323
- removed D8: 5V1, Diode_SMD:D_SOD-323
- removed D9: RED, LED_SMD:LED_0603_1608Metric
- removed J12, J14: BATT_2, Connector_PinHeader_2.54mm:PinHeader_2x02_P2.54mm_Vertical
- removed J13: PWR_1, Connector_PinHeader_2.54mm:PinHeader_2x02_P2.54mm_Vertical
- removed J15: PWR_3, Connector_PinHeader_2.54mm:PinHeader_1x08_P2.54mm_Vertical
- removed J16: CTL_3, Connector_PinHeader_2.54mm:PinHeader_1x08_P2.54mm_Vertical
- removed J17: CTL_1, Connector_PinHeader_2.54mm:PinHeader_2x02_P2.54mm_Vertical
- removed J18: CTL_2, Connector_PinHeader_2.54mm:PinHeader_2x02_P2.54mm_Vertical
- removed J19: PWR_4, Connector_PinHeader_2.54mm:PinHeader_1x04_P2.54mm_Vertical
- removed J20: CTL_5, Connector_PinHeader_2.54mm:PinHeader_1x04_P2.54mm_Vertical
- removed J21: CTL_4, Connector_PinHeader_2.00mm:PinHeader_1x09_P2.00mm_Vertical
- removed J22: INT_1, Connector_PinHeader_2.00mm:PinHeader_1x09_P2.00mm_Vertical
- removed Q4, Q5: BC817, Package_TO_SOT_SMD:SOT-23
- removed R37: 330R, Resistor_SMD:R_0402_1005Metric
- removed R38, R40: 2k2, Resistor_SMD:R_0402_1005Metric
- removed R39, R41, R43, R45, R47: 10k, Resistor_SMD:R_0402_1005Metric
- removed R42, R44: 68k, Resistor_SMD:R_0402_1005Metric
- removed R46: 20k, Resistor_SMD:R_0402_1005Metric
- removed R51: 100k, Resistor_SMD:R_0402_1005Metric
- removed R52, R53, R54: 1k, Resistor_SMD:R_0402_1005Metric
- removed TH1: NCP18XH103, Resistor_SMD:R_0603_1608Metric
- removed TP10: TP_BAT, TestPoint:TestPoint_Pad_D2.0mm
- removed TP2: TP_BTX, TestPoint:TestPoint_Pad_D2.0mm
- removed TP5: TP_USB_VDD, TestPoint:TestPoint_Pad_D2.0mm
- removed U3: MP1496, Package_TO_SOT_SMD:TSOT-23-8
- added C48: 22u, Capacitor_SMD:C_0805_2012Metric, F.Cu at (252.4, -12.8)
- added C49: 22u, Capacitor_SMD:C_0805_2012Metric, F.Cu at (241.1, -2.28)
- added C53: 100n, Capacitor_SMD:C_0402_1005Metric, F.Cu at (244.7, -3.82)
- added C54: 100n, Capacitor_SMD:C_0402_1005Metric, F.Cu at (237.7, 0.21)
- added C55: 10u, Capacitor_SMD:C_0805_2012Metric, F.Cu at (234.0, -0.15)
- added C56: 10u, Capacitor_SMD:C_0805_2012Metric, F.Cu at (243.4, -8.30)
- added C57: 100n, Capacitor_SMD:C_0402_1005Metric, F.Cu at (240.6, 0.21)
- added C58: 22u, Capacitor_SMD:C_0805_2012Metric, F.Cu at (241.1, -5.29)
- added C59: 470n, Capacitor_SMD:C_0402_1005Metric, F.Cu at (129.2, 3.63)
- added C60: 10u, Capacitor_SMD:C_0402_1005Metric, F.Cu at (126.3, 5.64)
- added C61: 22u, Capacitor_SMD:C_0805_2012Metric, F.Cu at (131.0, -9.51)
- added C62: 470n, Capacitor_SMD:C_0402_1005Metric, F.Cu at (136.0, -3.99)
- added C63: 470n, Capacitor_SMD:C_0402_1005Metric, F.Cu at (132.1, -1.05)
- added C64: 470n, Capacitor_SMD:C_0402_1005Metric, F.Cu at (129.2, 1.66)
- added C65: 10p, Capacitor_SMD:C_0402_1005Metric, F.Cu at (234.8, 42.2)
- added H7: MountingHole, MountingHole:MountingHole_2.1mm, F.Cu at (238.1, 26.5)
- added H8: MountingHole, MountingHole:MountingHole_2.1mm, F.Cu at (238.1, 32.2)
- added JP1: BootSelector, Jumper:SolderJumper-3_P2.0mm_Open_TrianglePad1.0x1.5mm, F.Cu at (193.8, 46.6)
- added U10: TP5100, Package_DFN_QFN:QFN-16-1EP_4x4mm_P0.65mm_EP2.1x2.1mm, F.Cu at (238.0, -11.2)
- added U11: STM32F411CEUx, Package_DFN_QFN:QFN-48-1EP_7x7mm_P0.5mm_EP5.6x5.6mm, B.Cu at (78.0, 120.0)
- added U12: HT7533-1-SOT89, Package_TO_SOT_SMD:SOT-89-3, F.Cu at (173.7, 20.1)
- added Y1: 7D024000H01, Crystal:Crystal_SMD_2016-4Pin_2.0x1.6mm, B.Cu at (77.5, 114.5)
- C10: value 22n -> 22u; footprint Capacitor_SMD:C_0402_1005Metric -> Capacitor_SMD:C_0805_2012Metric; moved to B.Cu
- C11: value 100n -> 2u2; footprint Capacitor_SMD:C_0402_1005Metric -> Capacitor_SMD:C_0603_1608Metric; moved to B.Cu
- C12: value 100n -> 22u; footprint Capacitor_SMD:C_0402_1005Metric -> Capacitor_SMD:C_0805_2012Metric; moved to B.Cu
- C13, C2, C26, C3, C5, C6, U6: moved to B.Cu
- C14: footprint Capacitor_SMD:C_0402_1005Metric -> Capacitor_SMD:C_0603_1608Metric; moved to B.Cu
- C15: value 22n -> 100n; footprint Capacitor_SMD:C_0402_1005Metric -> Capacitor_SMD:C_0603_1608Metric; moved to B.Cu
- C16, C17: value 4n7 -> 100n; footprint Capacitor_SMD:C_0402_1005Metric -> Capacitor_SMD:C_0603_1608Metric; moved to B.Cu
- C18: value 100n -> 1u; footprint Capacitor_SMD:C_0402_1005Metric -> Capacitor_SMD:C_0603_1608Metric
- C20: value 6n8 -> 22u; footprint Capacitor_SMD:C_0402_1005Metric -> Capacitor_SMD:C_0805_2012Metric
- C21: value 22u -> 22n; footprint Capacitor_SMD:C_0805_2012Metric -> Capacitor_SMD:C_0402_1005Metric; moved to B.Cu
- C22: value 6n8 -> 22n; moved to B.Cu
- C23, C24: value 22u -> 1u; footprint Capacitor_SMD:C_0805_2012Metric -> Capacitor_SMD:C_0603_1608Metric; moved to B.Cu
- C27: value 47u -> 22u; moved to B.Cu
- C28, C34: value 1u -> 22u; footprint Capacitor_SMD:C_0402_1005Metric -> Capacitor_SMD:C_0805_2012Metric
- C29, C30, C35: value 100n -> 22u; footprint Capacitor_SMD:C_0402_1005Metric -> Capacitor_SMD:C_0805_2012Metric
- C31: value 22u -> 27p; footprint Capacitor_SMD:C_0805_2012Metric -> Capacitor_SMD:C_0402_1005Metric
- C32: value 470n -> 22u; footprint Capacitor_SMD:C_0402_1005Metric -> Capacitor_SMD:C_0805_2012Metric
- C33: value 100n -> 27p
- C36: value 22u -> 470p; footprint Capacitor_SMD:C_0805_2012Metric -> Capacitor_SMD:C_0402_1005Metric
- C44: value 470n -> 470p
- C50: value 470n -> 22u; footprint Capacitor_SMD:C_0402_1005Metric -> Capacitor_SMD:C_0805_2012Metric; moved to F.Cu
- C51: value 22u -> 470n; footprint Capacitor_SMD:C_0805_2012Metric -> Capacitor_SMD:C_0402_1005Metric; moved to B.Cu
- C52: value 470n -> 10p
- C7: value 4u7 -> 22u; footprint Capacitor_SMD:C_0402_1005Metric -> Capacitor_SMD:C_0805_2012Metric
- C8: value 4u7 -> 22u; footprint Capacitor_SMD:C_0402_1005Metric -> Capacitor_SMD:C_0805_2012Metric; moved to B.Cu
- C9: value 22n -> 2u2; footprint Capacitor_SMD:C_0402_1005Metric -> Capacitor_SMD:C_0603_1608Metric; moved to B.Cu
- D1: value 3V3 -> SM4007PL; footprint Diode_SMD:D_SOD-323 -> Diode_SMD:D_SOD-123F; moved to B.Cu
- D2, D3: value 3V3 -> SB1045L; footprint Diode_SMD:D_SOD-323 -> Package_TO_SOT_SMD:TO-277B; moved to B.Cu
- D4: value PMEG045V100EPDAZ -> SS54; footprint rofi:D_SOT1289 -> Diode_SMD:D_SMA
- J1: value ESP_JTAG -> DEBUG; footprint Connector_PinHeader_2.54mm:PinHeader_2x05_P2.54mm_Vertical -> Connector_FFC-FPC:Hirose_FH12-10S-0.5SH_1x10-1MP_P0.50mm_Horizontal
- J10: value BATT_1 -> INTERFACE_CONN_TOP; footprint Connector_PinHeader_2.54mm:PinHeader_2x02_P2.54mm_Vertical -> rofi:2xM22-6550642R
- J11: value BATT_3 -> CONTROL_BOARD_CONN; footprint Connector_PinHeader_2.54mm:PinHeader_1x08_P2.54mm_Vertical -> Connector_PinHeader_2.00mm:PinHeader_2x12_P2.00mm_Vertical
- J3: value USB_ALT -> ROFICOMS; footprint Connector_PinHeader_2.54mm:PinHeader_1x04_P2.54mm_Vertical -> Connector_FFC-FPC:Hirose_FH12-20S-0.5SH_1x20-1MP_P0.50mm_Horizontal
- J4: value ShoeAConnectors -> MOTORS; footprint Connector_PinHeader_2.00mm:PinHeader_2x05_P2.00mm_Vertical -> Connector_FFC-FPC:Hirose_FH12-10S-0.5SH_1x10-1MP_P0.50mm_Horizontal
- J5: value MOTOR_BUS -> SHOE_B1; footprint Connector_PinHeader_2.00mm:PinHeader_1x04_P2.00mm_Vertical -> rofi:SlipRing-120220-0161
- J6: value MOTOR_BUS_ALT -> SHOE_B2; footprint Connector_PinHeader_2.00mm:PinHeader_1x03_P2.00mm_Vertical -> rofi:SlipRing-120220-0161
- J7: value ShoeBConnectors -> BATTERY_BOARD_CONN; footprint rofi:slipRingBrush -> Connector_PinHeader_2.00mm:PinHeader_2x12_P2.00mm_Vertical
- J8: value BIOS_SWD -> USB_C_Receptacle_USB2.0; footprint Connector_PinHeader_2.54mm:PinHeader_2x03_P2.54mm_Vertical -> rofi:USB_C_Female-16Pin-HPJF; moved to B.Cu
- J9: value USB_C_Receptacle_USB2.0 -> INTERFACE_CONN_BOTTOM; footprint rofi:USB_C_Female-16Pin-HPJF -> rofi:2xM22-6550642R
- L1, L2: value PA4548.152NLT -> 1u5/2u2; footprint rofi:PA4548 -> rofi:MGV1004; moved to B.Cu
- L3: value VLS3015CX-4R7M-1 -> 4u7; footprint rofi:VLS3015CX-1 -> rofi:SMNR5020
- L4: value SRN5020TA-5R6M -> 22u; footprint rofi:SRN5020TA -> rofi:SLO0630H; moved to F.Cu
- Q1, Q2: value SiA449DJ -> AONR21357; footprint Package_TO_SOT_SMD:Vishay_PowerPAK_SC70-6L_Single -> rofi:DFN3.3X3.3-EP; moved to F.Cu
- Q3: value SSM3K72CFS -> 2N7002; footprint Package_TO_SOT_SMD:SOT-416 -> Package_TO_SOT_SMD:SOT-23
- R1: value 100k -> 200k
- R10: value 10R -> 75k; moved to B.Cu
- R11, R12: value 56k -> 47k; moved to B.Cu
- R13, R15: value 6k8 -> 510k; moved to B.Cu
- R14: value 33k -> 56k; moved to B.Cu
- R16: value 40k2 -> 56k; moved to B.Cu
- R17: value 13k -> 10k
- R18: value 160R -> 470R; moved to F.Cu
- R19: value 10k -> 0R; moved to F.Cu
- R2: value 100k -> 10k; moved to B.Cu
- R20: value 261R -> 75m; footprint Resistor_SMD:R_0402_1005Metric -> Resistor_SMD:R_1206_3216Metric; moved to F.Cu
- R21: value 100R -> 68k; moved to F.Cu
- R22, R34: value 100k -> 10k; moved to F.Cu
- R23: value 50m -> 68k; footprint Resistor_SMD:R_1206_3216Metric -> Resistor_SMD:R_0402_1005Metric; moved to F.Cu
- R25, R26, R7: value 750k -> 100k
- R3: value 100k -> 150k; footprint Resistor_SMD:R_0402_1005Metric -> Capacitor_SMD:C_0402_1005Metric; moved to B.Cu
- R30, R32: moved to F.Cu
- R31: value 10k -> 20k; moved to F.Cu
- R33: value 10k -> 2k2; moved to F.Cu
- R35: value 100k -> 2k2; moved to F.Cu
- R36: value 330R -> 10k; moved to F.Cu
- R4: value 1k -> 150k; footprint Resistor_SMD:R_0402_1005Metric -> Capacitor_SMD:C_0402_1005Metric; moved to B.Cu
- R5: value 750k -> 0R; moved to B.Cu
- R56: value 1k -> 10k
- R6: value 1k -> 0R; moved to B.Cu
- R8: value 68k -> 31k6
- R9: value 68k -> 75k; moved to B.Cu
- SW1: value SW_Push -> SW_LEFT
- SW3: value SW_Push -> SW_MID
- SW5: value SW_Push -> SW_RIGHT
- TP1: value TP_BRX -> TP_BAT; moved to F.Cu
- U1, U2: value MP3431 -> Servo; footprint rofi:QFN-13 -> rofi:Dynamixel-XL-430-TOP
- U4: value MP2615 -> MT1470; footprint rofi:QFN-16 -> Package_TO_SOT_SMD:SOT-23-6; moved to F.Cu
- U5: value BQ29200 -> TPS61088; footprint Package_SON:Texas_S-PVSON-N8 -> rofi:VFQFN-20-4.5mmx3.5mm
- U7: value ICM-20948 -> MPU-6050; footprint Sensor_Motion:InvenSense_QFN-24_3x3mm_P0.4mm -> Sensor_Motion:InvenSense_QFN-24_4x4mm_P0.5mm
- U8: value CP2102N-A01-GQFN28 -> TPS61088; footprint Package_DFN_QFN:QFN-28-1EP_5x5mm_P0.5mm_EP3.35x3.35mm -> rofi:VFQFN-20-4.5mmx3.5mm
- U9: value STM32F030C8Tx -> PIEZO; footprint Package_QFP:LQFP-48_7x7mm_P0.5mm -> rofi:CST-931AP
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Connections:
- BT2 pad 2: /battery/GND -> B_GND
- C1 pad 1: /power/BATT_VDD -> C_BATT_VDD
- C1 pad 2: /power/GND -> C_GND
- C10 pad 1: Net-(C10-Pad1) -> USB_C_VDD
- C10 pad 2: /power/GND -> C_GND
- C11 pad 2: /power/GND -> C_GND
- C12 pad 1: Net-(C12-Pad1) -> C_BATT_VDD
- C12 pad 2: Net-(C12-Pad2) -> C_GND
- C13 pad 1: /power/BATT_VDD -> USB_C_VDD
- C13 pad 2: /power/GND -> C_GND
- C14 pad 1: Net-(C14-Pad1) -> C_BATT_VDD
- C14 pad 2: Net-(C14-Pad2) -> C_GND
- C15 pad 1: Net-(C15-Pad1) -> USB_C_VDD
- C15 pad 2: /power/GND -> C_GND
- C16 pad 2: /power/GND -> Net-(C16-Pad2)
- C17 pad 2: /power/GND -> Net-(C17-Pad2)
- C19 pad 1: Net-(C19-Pad1) -> B_3V3
- C19 pad 2: /power/GND -> B_GND
- C2 pad 1: /power/USB_C_VDD -> C_BATT_VDD
- C2 pad 2: /power/GND -> C_GND
- C20 pad 1: Net-(C20-Pad1) -> B_3V3
- C20 pad 2: Net-(C20-Pad2) -> B_GND
- C21 pad 2: /power/GND -> C_GND
- C22 pad 2: Net-(C22-Pad2) -> C_GND
- C23 pad 1: Net-(C19-Pad1) -> /power/BBV_OUTPUT
- C23 pad 2: /power/GND -> C_GND
- C24 pad 1: Net-(C21-Pad1) -> /power/UBV_OUTPUT
- C24 pad 2: /power/GND -> C_GND
- C25 pad 1: Net-(C19-Pad1) -> /control/3V3_ANALOG
- C25 pad 2: /power/GND -> C_GND
- C26 pad 1: Net-(C21-Pad1) -> /power/BBV_OUTPUT
- C26 pad 2: /power/GND -> C_GND
- C27 pad 1: /power/3V3 -> /power/UBV_OUTPUT
- C27 pad 2: /power/GND -> C_GND
- C28 pad 1: /battery/GND -> /power/BBV_OUTPUT
- C28 pad 2: Net-(C28-Pad2) -> C_GND
- C29 pad 1: Net-(C29-Pad1) -> /power/UBV_OUTPUT
- C29 pad 2: Net-(C29-Pad2) -> C_GND
- C3 pad 1: /power/BATT_VDD -> USB_C_VDD
- C3 pad 2: /power/GND -> C_GND
- C30 pad 1: Net-(C29-Pad2) -> /power/BBV_OUTPUT
- C30 pad 2: /battery/GND -> C_GND
- C31 pad 1: /battery/GND -> Net-(C31-Pad1)
- C31 pad 2: /battery/INT -> C_GND
- C32 pad 1: Net-(C32-Pad1) -> /power/UBV_OUTPUT
- C32 pad 2: /battery/GND -> C_GND
- C33 pad 2: Net-(C33-Pad2) -> C_GND
- C34 pad 1: Net-(C34-Pad1) -> /power/BBV_OUTPUT
- C34 pad 2: /battery/GND -> C_GND
- C35 pad 1: /battery/BAT+ -> /power/UBV_OUTPUT
- C35 pad 2: /battery/GND -> C_GND
- C36 pad 1: /battery/BAT+ -> Net-(C36-Pad1)
- C36 pad 2: /battery/GND -> C_GND
- C37 pad 2: /battery/PWR_START -> B_PWR_START
- C38 pad 1: /battery/PWR_SHUTDOWN -> B_PWR_SHUTDOWN
- C38 pad 2: /battery/GND -> B_GND
- C39 pad 1: /bios/3V3 -> C_3V3
- C39 pad 2: /bios/GND -> C_GND
- C4 pad 1: /power/USB_C_VDD -> B_BATT_VDD
- C4 pad 2: /power/GND -> B_GND
- C40 pad 1: /bios/3V3 -> C_3V3
- C40 pad 2: /bios/GND -> C_GND
- C41 pad 1: /bios/3V3 -> C_GND
- C41 pad 2: /bios/GND -> C_3V3
- C42 pad 1: /bios/3V3 -> C_GND
- C42 pad 2: /bios/GND -> C_3V3
- C43 pad 1: /bios/GND -> C_GND
- C44 pad 1: ESP_EN -> Net-(C44-Pad1)
- C44 pad 2: /bios/GND -> C_GND
- C45 pad 1: /interface/SW_LEFT -> I_SW_LEFT
- C45 pad 2: /interface/GND -> I_GND
- C46 pad 1: /interface/SW_MID -> I_SW_MID
- C46 pad 2: /interface/GND -> I_GND
- C47 pad 1: /interface/SW_RIGHT -> I_SW_RIGHT
- C47 pad 2: /interface/GND -> I_GND
- C5 pad 1: /power/BATT_VDD -> C_BATT_VDD
- C5 pad 2: /power/GND -> C_GND
- C50 pad 1: /bios/3V3 -> B_INT
- C50 pad 2: /bios/GND -> B_GND
- C51 pad 1: /bios/3V3 -> C_GND
- C51 pad 2: /bios/GND -> Net-(C51-Pad2)
- C52 pad 1: /bios/3V3 -> Net-(C52-Pad1)
- C52 pad 2: /bios/GND -> C_GND
- C6 pad 1: /power/USB_C_VDD -> USB_C_VDD
- C6 pad 2: /power/GND -> C_GND
- C7 pad 1: Net-(C7-Pad1) -> B_BATT_VDD
- C7 pad 2: /power/GND -> B_GND
- C8 pad 1: Net-(C8-Pad1) -> C_BATT_VDD
- C8 pad 2: /power/GND -> C_GND
- C9 pad 2: /power/GND -> C_GND
- D1 pad 1: /power/USB_TO_BUS_EN -> Net-(D1-Pad1)
- D1 pad 2: /power/GND -> BATT_TO_BUS_EN
- D14 pad 1: /battery/CHG_OK -> B_CHG_OK
- D16 pad 1: /power/GND -> C_GND
- D17 pad 1: /power/GND -> C_GND
- D18 pad 1: /power/GND -> C_GND
- D2 pad 1: /power/BATT_TO_BUS_EN -> /power/BBV_OUTPUT
- D2 pad 2: /power/GND -> /power/BBV_OUTPUT
- D3 pad 1: Net-(D3-Pad1) -> /power/UBV_OUTPUT
- D3 pad 2: /power/GND -> /power/UBV_OUTPUT
- D4 pad 1: /power/INT -> Net-(C54-Pad1)
- D4 pad 2: Net-(C19-Pad1) -> B_GND
- J1 pad 1: /bios/3V3 -> C_GND
- J1 pad 10: (no net) -> C_GND
- J1 pad 3: /bios/GND -> ESP_TCK
- J1 pad 4: ESP_TCK -> ESP_TDO
- J1 pad 5: /bios/GND -> ESP_TDI
- J1 pad 6: ESP_TDO -> SWCLK
- J1 pad 7: /bios/GND -> SWDIO
- J1 pad 8: ESP_TDI -> SWRST
- J1 pad 9: /bios/GND -> C_3V3
- J10 pad 1: /battery/BAT_VDD -> I_PIEZO_P
- J10 pad 2: /battery/BAT_VDD -> I_PIEZO_N
- J10 pad 3: /battery/GND -> I_CHG_EN
- J10 pad 4: /battery/GND -> I_CHG_OK
- J11 pad 1: /battery/INT -> C_BUZZER_P
- J11 pad 2: /battery/CHG_EN -> C_BUZZER_N
- J11 pad 3: /battery/BATT_VOLTAGE -> C_CHG_EN
- J11 pad 4: /battery/PWR_SHUTDOWN -> C_CHG_OK
- J11 pad 5: /battery/PWR_START -> C_PWR_SHUTDOWN
- J11 pad 6: /battery/3V3 -> (no net)
- J11 pad 7: /battery/CHG_AC_OK -> C_SW_RIGHT
- J11 pad 8: /battery/CHG_OK -> C_SW_MID
- J2 pad 1: /interface/SDA -> I_SDA
- J2 pad 2: /interface/SCL -> I_SCL
- J2 pad 3: /interface/3V3 -> I_3V3
- J2 pad 4: /interface/GND -> I_GND
- J3 pad 1: /bios/GND -> C_GND
- J3 pad 2: USB_C_D- -> SPI_SCK
- J3 pad 3: USB_C_D+ -> C_GND
- J3 pad 4: /bios/USB_C_VDD -> SPI_MISO_MOSI
- J4 pad 1: /control/BATT_VDD -> MOTORS_TX
- J4 pad 10: /bios/GND -> C_GND
- J4 pad 2: DOCK_3_CE -> MOTORS_RX
- J4 pad 3: /bios/INT -> C_GND
- J4 pad 4: DOCK_2_CE -> C_BATT_VDD
- J4 pad 5: /control/EXT -> C_BATT_VDD
- J4 pad 6: DOCK_1_CE -> C_BATT_VDD
- J4 pad 7: SPI_SCK -> C_GND
- J4 pad 8: SPI_MISO_MOSI -> C_GND
- J4 pad 9: /bios/GND -> C_GND
- J5 pad 1: /bios/GND -> C_GND
- J5 pad 2: /control/BATT_VDD -> SPI_SCK
- J5 pad 3: MOTORS_RX -> C_GND
- J5 pad 4: MOTORS_TX -> SPI_MISO_MOSI
- J6 pad 1: /bios/GND -> C_GND
- J6 pad 2: /control/BATT_VDD -> /control/EXT
- J6 pad 3: MOTORS_TX -> C_INT
- J7 pad 1: /bios/GND -> B_PIEZO_P
- J7 pad 10: DOCK_5_CE -> (no net)
- J7 pad 11: DOCK_6_CE -> (no net)
- J7 pad 12: /bios/GND -> B_3V3
- J7 pad 2: /control/BATT_VDD -> B_PIEZO_N
- J7 pad 3: MOTORS_RX -> B_CHG_EN
- J7 pad 4: MOTORS_TX -> B_CHG_OK
- J7 pad 5: /bios/INT -> B_PWR_SHUTDOWN
- J7 pad 6: /control/EXT -> B_PWR_START
- J7 pad 7: SPI_SCK -> (no net)
- J7 pad 8: SPI_MISO_MOSI -> (no net)
- J7 pad 9: DOCK_4_CE -> (no net)
- L1 pad 1: /power/BATT_VDD -> Net-(C16-Pad2)
- L1 pad 2: Net-(C12-Pad2) -> C_BATT_VDD
- L2 pad 1: /power/USB_C_VDD -> Net-(C17-Pad2)
- L2 pad 2: Net-(C14-Pad2) -> USB_C_VDD
- L3 pad 2: /power/3V3 -> B_3V3
- L4 pad 2: Net-(C33-Pad1) -> Net-(C54-Pad1)
- Q1 pad 1: /battery/BAT+ -> Net-(Q1-Pad1)
- Q1 pad 3: /battery/GND -> /battery/BAT+
- Q2 pad 1: Net-(Q1-Pad4) -> Net-(Q1-Pad1)
- Q2 pad 3: Net-(C37-Pad1) -> B_BATT_VDD
- Q3 pad 1: /battery/PWR_SHUTDOWN -> B_PWR_SHUTDOWN
- Q3 pad 2: /battery/GND -> B_GND
- R1 pad 1: /power/BATT_TO_BUS_EN -> B_BATT_VDD
- R1 pad 2: /power/BATT_VDD -> Net-(R1-Pad2)
- R10 pad 1: Net-(C18-Pad1) -> Net-(R10-Pad1)
- R10 pad 2: Net-(R10-Pad2) -> C_GND
- R11 pad 1: Net-(C16-Pad1) -> Net-(C31-Pad1)
- R11 pad 2: /power/GND -> Net-(C36-Pad1)
- R12 pad 1: Net-(C17-Pad1) -> Net-(C33-Pad1)
- R12 pad 2: /power/GND -> Net-(C44-Pad1)
- R13 pad 1: Net-(C20-Pad1) -> /power/BBV_OUTPUT
- R13 pad 2: /power/GND -> /power/BBV_FB
- R14 pad 1: Net-(R14-Pad1) -> /power/BBV_FB
- R14 pad 2: Net-(R14-Pad2) -> C_GND
- R15 pad 1: Net-(C22-Pad1) -> /power/UBV_OUTPUT
- R15 pad 2: /power/GND -> /power/UBV_FB
- R16 pad 1: /power/3V3 -> /power/UBV_FB
- R16 pad 2: Net-(R14-Pad1) -> C_GND
- R17 pad 1: Net-(R14-Pad1) -> Net-(D16-Pad2)
- R17 pad 2: /power/GND -> C_BATT_VDD
- R18 pad 1: Net-(C29-Pad1) -> Net-(D14-Pad2)
- R18 pad 2: /battery/BAT+ -> B_3V3
- R19 pad 2: Net-(C28-Pad2) -> B_GND
- R2 pad 1: /power/USB_TO_BUS_EN -> Net-(C11-Pad1)
- R2 pad 2: /power/USB_C_VDD -> USB_TO_BUS_EN
- R20 pad 1: Net-(C29-Pad2) -> /battery/BAT+
- R20 pad 2: Net-(BT1-Pad2) -> Net-(C54-Pad1)
- R21 pad 1: Net-(R21-Pad1) -> C_INT
- R21 pad 2: Net-(BT1-Pad2) -> /control/BUS_VOLTAGE
- R22 pad 1: Net-(R22-Pad1) -> /control/BUS_VOLTAGE
- R22 pad 2: Net-(D6-Pad1) -> C_GND
- R23 pad 1: /battery/BAT+ -> USB_C_VDD
- R23 pad 2: Net-(L4-Pad1) -> /control/USB_VOLTAGE
- R24 pad 2: Net-(Q1-Pad4) -> Net-(Q1-Pad1)
- R25 pad 2: /battery/PWR_START -> B_PWR_START
- R26 pad 1: /battery/PWR_SHUTDOWN -> B_PWR_SHUTDOWN
- R26 pad 2: /battery/GND -> B_GND
- R27 pad 1: /battery/3V3 -> B_3V3
- R27 pad 2: /battery/PWR_SHUTDOWN -> B_PWR_SHUTDOWN
- R28 pad 1: /bios/3V3 -> C_3V3
- R28 pad 2: BIOS_SDA -> C_SDA
- R29 pad 1: BIOS_SCL -> C_SCL
- R29 pad 2: /bios/3V3 -> C_3V3
- R3 pad 1: Net-(D3-Pad1) -> Net-(R3-Pad1)
- R3 pad 2: /power/BATT_VDD -> Net-(C16-Pad2)
- R30 pad 1: Net-(Q4-Pad1) -> /control/USB_VOLTAGE
- R30 pad 2: DTR -> C_GND
- R31 pad 1: Net-(Q5-Pad1) -> C_BATT_VDD
- R31 pad 2: RTS -> /control/BATT_VOLTAGE
- R32 pad 1: Net-(Q5-Pad1) -> /control/BATT_VOLTAGE
- R32 pad 2: /bios/3V3 -> C_GND
- R33 pad 1: /bios/3V3 -> QC_2_M
- R33 pad 2: ESP_EN -> USB_C_D-
- R34 pad 1: Net-(D8-Pad1) -> USB_C_D-
- R34 pad 2: Net-(D7-Pad1) -> QC_10_N
- R35 pad 1: /bios/3V3 -> QC_2_P
- R35 pad 2: USB_BRIDGE_EN -> USB_C_D+
- R36 pad 1: /bios/3V3 -> USB_C_D+
- R36 pad 2: Net-(D9-Pad2) -> QC_10_P
- R4 pad 1: Net-(C16-Pad1) -> Net-(R4-Pad1)
- R4 pad 2: Net-(R4-Pad2) -> Net-(C17-Pad2)
- R5 pad 1: Net-(C19-Pad1) -> Net-(R5-Pad1)
- R5 pad 2: Net-(R5-Pad2) -> C_GND
- R55 pad 2: /power/3V3 -> C_3V3
- R56 pad 2: /power/INT -> C_INT
- R6 pad 1: Net-(C17-Pad1) -> Net-(R6-Pad1)
- R6 pad 2: Net-(R6-Pad2) -> C_GND
- R7 pad 1: Net-(C21-Pad1) -> B_3V3
- R8 pad 1: /power/GND -> Net-(R7-Pad2)
- R8 pad 2: Net-(R5-Pad2) -> B_GND
- R9 pad 1: /power/GND -> Net-(R9-Pad1)
- R9 pad 2: Net-(R7-Pad2) -> C_GND
- SW1 pad 1: /interface/SW_LEFT -> I_SW_LEFT
- SW1 pad 2: /interface/GND -> I_GND
- SW2 pad 1: /interface/STOP_BUTTON -> I_STOP_SW
- SW2 pad 2: /interface/GND -> I_GND
- SW3 pad 1: /interface/SW_MID -> I_SW_MID
- SW3 pad 2: /interface/GND -> I_GND
- SW4 pad 1: /interface/START_BUTTON -> I_START_SW
- SW4 pad 2: /interface/GND -> I_GND
- SW5 pad 1: /interface/SW_RIGHT -> I_SW_RIGHT
- SW5 pad 2: /interface/GND -> I_GND
- TP1 pad 1: BIOS_RX -> C_BATT_VDD
- TP3 pad 1: BIOS_SDA -> C_SDA
- TP4 pad 1: BIOS_SCL -> C_SCL
- TP6 pad 1: /power/INT -> C_INT
- U4 pad 1: Net-(C33-Pad1) -> B_GND
- U4 pad 2: /battery/INT -> Net-(C18-Pad2)
- U4 pad 3: Net-(C28-Pad2) -> B_BATT_VDD
- U4 pad 4: /battery/GND -> Net-(R7-Pad2)
- U4 pad 5: /battery/GND -> Net-(R1-Pad2)
- U4 pad 6: Net-(R22-Pad1) -> Net-(C18-Pad1)
- U5 pad 1: Net-(C29-Pad1) -> Net-(C9-Pad1)
- U5 pad 2: Net-(C29-Pad2) -> Net-(D1-Pad1)
- U5 pad 3: Net-(R21-Pad1) -> Net-(R3-Pad1)
- U5 pad 4: Net-(C32-Pad1) -> Net-(C16-Pad2)
- U5 pad 5: /battery/GND -> Net-(C16-Pad2)
- U5 pad 6: /battery/GND -> Net-(C16-Pad2)
- U5 pad 7: /battery/BAT+ -> Net-(C16-Pad2)
- U5 pad 8: Net-(U5-Pad8) -> Net-(C16-Pad1)
- U5 pad 9: /battery/GND -> C_BATT_VDD
- U6 pad 1: /bios/GND -> C_GND
- U6 pad 15: /bios/GND -> C_GND
- U6 pad 2: /bios/3V3 -> C_3V3
- U6 pad 24: MOTORS_RX -> DOCK_4_CE
- U6 pad 25: IO0 -> ESP_BOOT
- U6 pad 29: SPI_SCK -> BIOS_RX
- U6 pad 30: SPI_MISO_MOSI -> SPI_SCK
- U6 pad 31: BIOS_RX -> SPI_MISO_MOSI
- U6 pad 33: BIOS_TX -> MOTORS_RX
- U6 pad 36: BIOS_SDA -> C_SDA
- U6 pad 37: BIOS_SCL -> C_SCL
- U6 pad 38: /bios/GND -> C_GND
- U6 pad 39: /bios/GND -> C_GND
- U6 pad 7: DOCK_4_CE -> BIOS_TX
- U7 pad 1: (no net) -> C_GND
- U7 pad 11: /bios/GND -> C_GND
- U7 pad 12: (no net) -> MPU_INT
- U7 pad 13: /bios/3V3 -> C_3V3
- U7 pad 18: /bios/GND -> C_GND
- U7 pad 20: /bios/GND -> Net-(C51-Pad2)
- U7 pad 22: /bios/3V3 -> (no net)
- U7 pad 23: BIOS_SCL -> C_SCL
- U7 pad 24: BIOS_SDA -> C_SDA
- U7 pad 8: /bios/3V3 -> C_3V3
- U7 pad 9: Net-(R51-Pad1) -> C_GND
- U8 pad 1: (no net) -> Net-(C11-Pad1)
- U8 pad 10: (no net) -> Net-(C22-Pad1)
- U8 pad 11: (no net) -> C_GND
- U8 pad 12: USB_SUSPEND -> C_GND
- U8 pad 13: (no net) -> Net-(R6-Pad1)
- U8 pad 14: (no net) -> /power/UBV_OUTPUT
- U8 pad 15: (no net) -> /power/UBV_OUTPUT
- U8 pad 16: (no net) -> /power/UBV_OUTPUT
- U8 pad 17: (no net) -> /power/UBV_FB
- U8 pad 18: Net-(D10-Pad1) -> Net-(C33-Pad1)
- U8 pad 19: Net-(D9-Pad1) -> Net-(R10-Pad1)
- U8 pad 2: USB_CLK -> USB_TO_BUS_EN
- U8 pad 20: (no net) -> C_GND
- U8 pad 21: (no net) -> C_GND
- U8 pad 3: /bios/GND -> Net-(R4-Pad1)
- U8 pad 4: USB_C_D+ -> Net-(C17-Pad2)
- U8 pad 5: USB_C_D- -> Net-(C17-Pad2)
- U8 pad 6: /bios/3V3 -> Net-(C17-Pad2)
- U8 pad 7: /bios/3V3 -> Net-(C17-Pad2)
- U8 pad 8: Net-(D8-Pad1) -> Net-(C17-Pad1)
- U8 pad 9: USB_BRIDGE_EN -> USB_C_VDD
- U9 pad 1: /bios/3V3 -> B_PIEZO_P
- U9 pad 2: /bios/CHG_OK -> B_PIEZO_N
Routing:
- net /bios/3V3: track 185.3 -> 0.00 mm, vias 11 -> 0
- net MOTORS_TX: track 121.7 -> 0.00 mm, vias 3 -> 0
- net MOTORS_RX: track 116.1 -> 0.00 mm, vias 3 -> 0
- net /power/USB_C_VDD: track 114.5 -> 0.00 mm, vias 3 -> 0
- net BIOS_SCL: track 106.1 -> 0.00 mm, vias 8 -> 0
- net /power/INT: track 101.5 -> 0.00 mm, vias 2 -> 0
- net SPI_MISO_MOSI: track 101.3 -> 0.00 mm, vias 1 -> 0
- net BIOS_SDA: track 96.8 -> 0.00 mm, vias 3 -> 0
- net SPI_SCK: track 94.4 -> 0.00 mm, vias 1 -> 0
- net /power/BATT_TO_BUS_EN: track 93.1 -> 0.00 mm
- net /bios/USB_C_VDD: track 91.3 -> 0.00 mm, vias 7 -> 0
- net /bios/PWR_SHUTDOWN: track 87.8 -> 0.00 mm, vias 4 -> 0
- net DOCK_3_CE: track 86.0 -> 0.00 mm, vias 1 -> 0
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- removed copper zone on B.Cu, net /battery/BAT+
- removed copper zone on B.Cu, net /battery/BAT_VDD
- removed copper zone on B.Cu, net /battery/GND
- removed copper zone on F.Cu, net /battery/GND
- removed copper zone on B.Cu, net /battery/INT
- removed copper zone on F.Cu, net /bios/3V3
- removed copper zone on B.Cu, net /bios/GND
- removed copper zone on F.Cu, net /bios/GND
- removed copper zone on B.Cu, net /bios/USB_C_VDD
- removed copper zone on F.Cu, net /bios/USB_C_VDD
- removed copper zone on B.Cu, net /interface/GND
- removed copper zone on F.Cu, net /interface/GND
- removed copper zone on F.Cu, net /power/3V3
- removed copper zone on F.Cu, net /power/BATT_VDD
- removed copper zone on B.Cu, net /power/GND
- removed copper zone on F.Cu, net /power/GND
- removed copper zone on F.Cu, net /power/USB_C_VDD
- removed copper zone on F.Cu, net Net-(C12-Pad2)
- removed copper zone on F.Cu, net Net-(C14-Pad2)
- removed copper zone on B.Cu, net Net-(C18-Pad2)
- removed copper zone on F.Cu, net Net-(C18-Pad2)
- removed copper zone on F.Cu, net Net-(C19-Pad1)
- removed copper zone on F.Cu, net Net-(C21-Pad1)
- removed copper zone on B.Cu, net Net-(Q1-Pad4)
Other:
- board size 245.9 x 74 mm -> 193.5 x 76 mm
- copper layers 2 -> 4
- net class Default: clearance 0.15 -> 0.127; via_dia 0.8 -> 0.45; via_drill 0.4 -> 0.2
- rule trace_clearance: 0.15 -> 0.127
- rule trace_min: 0.15 -> 0.127
- rule via_min_drill: 0.3 -> 0.2
- rule via_min_size: 0.6 -> 0.45
- board text removed: "3V3"
- board text removed: "BATT"
- board text removed: "CHG_ACT"
- board text removed: "CHG_PWR"
- board text removed: "E3 E2 E1 DA G VD IN EX CK G"
- board text removed: "GND VDD MRX MTX INT EXT SCK DAT CE4 CE5 CE6 GND"
- board text removed: "GND VDD RX TX"
- board text removed: "INT"
- board text removed: "IO 3V G CL RS G"
- board text removed: "RX TX SDA SCL"
- board text removed: "RoFI Universal Module - Battery Board v0.1 11/2019"
- board text removed: "RoFI Universal Module - Control Board v0.1 11/2019"
- board text removed: "RoFI Universal Module - Power Board v0.1 11/2019"
- board text removed: "RoFI Universal Module UI Board v0.1 11/2019"
- board text removed: "TMS TCK TDO TDI"
- board text removed: "USB"

Commit message: universalModule: Prepare electronics v0.2
Parts:
- removed C2, C3, C50: 22u, Capacitor_SMD:C_0805_2012Metric
- removed C40: 470n, Capacitor_SMD:C_0402_1005Metric
- removed C56: 10u, Capacitor_SMD:C_0805_2012Metric
- added BODY1: BOARD, kikit:Board, F.Cu at (207.5, 167.0)
- added BODY2: BOARD, kikit:Board, F.Cu at (39.7, 185.0)
- added BODY3: BOARD, kikit:Board, F.Cu at (117.5, 167.1)
- added BODY4: BOARD, kikit:Board, F.Cu at (178.7, 106.0)
- added BODY5: BOARD, kikit:Board, F.Cu at (305.4, 167.0)
- added CABLE1: BOARD, kikit:Board, F.Cu at (155.7, 66.2)
- added CABLE2: BOARD, kikit:Board, F.Cu at (233.2, 136.2)
- added DEBUG1: BOARD, kikit:Board, F.Cu at (81.4, 100.0)
- added H10: MountingHole, MountingHole:MountingHole_2.7mm, F.Cu at (196.0, 142.0)
- added H11: MountingHole, MountingHole:MountingHole_2.7mm, F.Cu at (184.0, 118.0)
- added H12: MountingHole, MountingHole:MountingHole_2.7mm, F.Cu at (196.0, 118.0)
- added H13: MountingHole, rofi:RoFICoM-MountingHolesThreaded, F.Cu at (205.0, 60.0)
- added H14: MountingHole, rofi:RoFICoM-MountingHolesThreaded, F.Cu at (270.0, 60.0)
- added H15: MountingHole, rofi:RoFICoM-MountingHolesThreaded, F.Cu at (105.0, 60.0)
- added H16: MountingHole, rofi:ThreadedHole-M2, F.Cu at (189.5, 37.4)
- added H17: MountingHole, rofi:ThreadedHole-M2, F.Cu at (182.3, 44.3)
- added H18: MountingHole, rofi:ThreadedHole-M2, F.Cu at (182.3, 75.7)
- added H19: MountingHole, rofi:ThreadedHole-M2, F.Cu at (189.5, 82.6)
- added H20: MountingHole, rofi:ThreadedHole-M2, F.Cu at (220.5, 82.6)
- added H21: MountingHole, rofi:ThreadedHole-M2, F.Cu at (227.8, 75.7)
- added H22: MountingHole, rofi:ThreadedHole-M2, F.Cu at (227.8, 44.3)
- added H23: MountingHole, rofi:ThreadedHole-M2, F.Cu at (220.5, 37.4)
- added H24: MountingHole, rofi:ThreadedHole-M2, F.Cu at (252.0, 35.8)
- added H25: MountingHole, rofi:ThreadedHole-M2, F.Cu at (247.2, 44.5)
- added H26: MountingHole, rofi:ThreadedHole-M2, F.Cu at (247.2, 75.5)
- added H27: MountingHole, rofi:ThreadedHole-M2, F.Cu at (252.0, 84.2)
- added H28: MountingHole, rofi:ThreadedHole-M2, F.Cu at (123.0, 35.8)
- added H29: MountingHole, rofi:ThreadedHole-M2, F.Cu at (127.8, 44.5)
- added H30: MountingHole, rofi:ThreadedHole-M2, F.Cu at (127.8, 75.5)
- added H31: MountingHole, rofi:ThreadedHole-M2, F.Cu at (123.0, 84.2)
- added H9: MountingHole, MountingHole:MountingHole_2.7mm, F.Cu at (184.0, 142.0)
- added J12: SHOE, Connector_FFC-FPC:Hirose_FH12-24S-0.5SH_1x24-1MP_P0.50mm_Horizontal, F.Cu at (195.0, 130.0)
- added J13: SLIP_RING_OUT, Connector_FFC-FPC:Hirose_FH12-40S-0.5SH_1x40-1MP_P0.50mm_Horizontal, B.Cu at (285.1, 205.0)
- added J14: REFERENCE_PINS, rofi:SlipRing-120220-0161, F.Cu at (304.3, 189.0)
- added J15: INPUT, rofi:UM_SHOE_PADS, F.Cu at (118.9, 60.0)
- added J16: ST-LINK A, Connector_IDC:IDC-Header_2x05_P2.54mm_Vertical, F.Cu at (105.0, 135.0)
- added J17: ST-LINK_B, Connector_IDC:IDC-Header_2x05_P2.54mm_Vertical, F.Cu at (85.0, 135.0)
- added J18: Conn_02x10_Odd_Even, Connector_PinSocket_2.54mm:PinSocket_2x10_P2.54mm_Vertical, F.Cu at (125.0, 115.0)
- added J19: ESP-DBG, Connector_IDC:IDC-Header_2x05_P2.54mm_Vertical, F.Cu at (105.0, 110.0)
- added J20: Conn_ST_STDC14, Connector_PinSocket_1.27mm:PinSocket_2x07_P1.27mm_Vertical_SMD, F.Cu at (86.0, 115.0)
- added J21: DEBUG, Connector_FFC-FPC:Hirose_FH12-10S-0.5SH_1x10-1MP_P0.50mm_Horizontal, F.Cu at (140.0, 126.5)
- added J22: SHOE_OUT, rofi:Hirose_FH12-40S-0.5SH_1x40-1MP_P0.50mm_Horizontal, F.Cu at (98.7, 205.1)
- added J23: ROFICOM1_A, rofi:SOLO-9258, F.Cu at (105.0, 42.0)
- added J24: DBG1, Connector_PinHeader_2.54mm:PinHeader_1x07_P2.54mm_Vertical, F.Cu at (112.0, 35.0)
- added J25: ROFICOM1_B, rofi:SOLO-9258, F.Cu at (105.0, 72.0)
- added J26: ROFICOM1_C, rofi:SOLO-9258, F.Cu at (105.0, 78.0)
- added J27: OUTPUT, rofi:UM_SHOE_PADS, F.Cu at (127.0, 60.0)
- added J28: INPUT, rofi:UM_SHOE_PADS, F.Cu at (248.0, 60.0)
- added J29: ROFICOM1_A, rofi:SOLO-9258, F.Cu at (270.0, 42.0)
- added J30: DBG1, Connector_PinHeader_2.54mm:PinHeader_1x07_P2.54mm_Vertical, F.Cu at (278.0, 35.0)
- added J31: ROFICOM1_B, rofi:SOLO-9258, F.Cu at (270.0, 72.0)
- added J32: ROFICOM1_C, rofi:SOLO-9258, F.Cu at (270.0, 78.0)
- added J33: OUTPUT, rofi:UM_SHOE_PADS, F.Cu at (254.0, 60.0)
- added J34: INPUT, rofi:UM_SHOE_PADS, F.Cu at (184.0, 60.0)
- added J35: ROFICOM1_A, rofi:SOLO-9258, F.Cu at (205.0, 42.0)
- added J36: DBG1, Connector_PinHeader_2.54mm:PinHeader_1x07_P2.54mm_Vertical, F.Cu at (212.0, 35.0)
- added J37: ROFICOM1_B, rofi:SOLO-9258, F.Cu at (205.0, 78.0)
- added J38: ROFICOM1_C, rofi:SOLO-9258, F.Cu at (205.0, 72.0)
- added J39: OUTPUT, rofi:UM_SHOE_PADS, F.Cu at (226.0, 60.0)
- added J40: A, rofi:UM_SHOE_PADS_BOTH, F.Cu at (153.0, 60.0)
- added J41: B, rofi:UM_SHOE_PADS_BOTH, F.Cu at (162.0, 60.0)
- added J42: SHOE, rofi:FPC_0.5_24_PADS, B.Cu at (217.5, 130.0)
- added J43: B, rofi:UM_SHOE_PADS_BOTH, F.Cu at (254.0, 129.9)
- added R37: 5k1, Resistor_SMD:R_0402_1005Metric, B.Cu at (92.7, 195.8)
- added R38: 5k1, Resistor_SMD:R_0402_1005Metric, B.Cu at (92.7, 191.8)
- added SHOE1: BOARD, kikit:Board, F.Cu at (105.7, 33.0)
- added SHOE2: BOARD, kikit:Board, F.Cu at (201.8, 33.0)
- added SHOE3: BOARD, kikit:Board, F.Cu at (262.9, 33.0)
- added U3: Servo, rofi:Dynamixel-XL-430-TOP, F.Cu at (305.0, 205.0)
- C1, C25, C52, C59, C60, C61, C62, C63, C64, C65, D16, D17, D18, J10, R17, R21, R22, R23, R28, R29, R30, R31, R32, R33, R34, R35, R36, R55, R56, U12: moved to B.Cu
- J1: footprint Connector_FFC-FPC:Hirose_FH12-10S-0.5SH_1x10-1MP_P0.50mm_Horizontal -> rofi:Hirose_FH12-10S-0.5SH_1x10-1MP_P0.50mm_Horizontal
- J11: footprint Connector_PinHeader_2.00mm:PinHeader_2x12_P2.00mm_Vertical -> Connector_PinHeader_2.00mm:PinHeader_2x12_P2.00mm_Vertical_SMD; moved to B.Cu
- J3: value ROFICOMS -> BOARD_IN; footprint Connector_FFC-FPC:Hirose_FH12-20S-0.5SH_1x20-1MP_P0.50mm_Horizontal -> Connector_FFC-FPC:Hirose_FH12-40S-0.5SH_1x40-1MP_P0.50mm_Horizontal
- J4: value MOTORS -> SERVO; footprint Connector_FFC-FPC:Hirose_FH12-10S-0.5SH_1x10-1MP_P0.50mm_Horizontal -> Connector_PinHeader_2.54mm:PinHeader_1x03_P2.54mm_Vertical
- J6: footprint rofi:SlipRing-120220-0161 -> rofi:SlipRing-120220-0161-incomplete
- J9: footprint rofi:2xM22-6550642R -> rofi:2xM22-6550642R-MIRRORED; moved to B.Cu
- R24, TP3, TP4: moved to F.Cu
- R8: value 31k6 -> 22k
- U4: value MT1470 -> SD8942
- moved D16 258.9 mm to (81.7, 208.9), turned to 270 degrees
- moved H8 246.2 mm to (96.2, 233.5)
- moved TP6 244.3 mm to (145.9, 226.6)
- moved R7 242.6 mm to (192.9, 211.3), turned to 270 degrees
- moved Q3 242.4 mm to (186.6, 222.4), turned to 90 degrees
- moved R8 241.9 mm to (192.9, 213.6), turned to 270 degrees
- moved C18 241.1 mm to (187.9, 212.9), turned to 90 degrees
- moved L3 239.7 mm to (184.1, 210.9), turned to 270 degrees
- moved R27 237.3 mm to (183.1, 225.3), turned to 90 degrees
- moved C4 237.2 mm to (189.0, 206.8), turned to 90 degrees
- moved C20 237.1 mm to (184.2, 205.6), turned to 90 degrees
- moved R56 237.0 mm to (83.0, 202.1), turned to 270 degrees
- moved D18 236.3 mm to (81.6, 202.1), turned to 90 degrees
- moved Q2 235.9 mm to (183.0, 216.0), turned to 90 degrees
- moved U4 235.3 mm to (190.6, 212.4), turned to 90 degrees
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Connections:
- net Net-(BT1-Pad2) renamed /battery/BATT_MID
- J1 pad 1: C_GND -> ESP_EN
- J3 pad 1: C_GND -> /servoBoard/GND
- J3 pad 10: C_BATT_VDD -> /servoBoard/MOTORS_TX
- J3 pad 11: C_BATT_VDD -> (no net)
- J3 pad 12: C_GND -> /servoBoard/GND
- J3 pad 13: C_GND -> /servoBoard/GND
- J3 pad 14: C_INT -> /servoBoard/BATT_VDD
- J3 pad 15: C_INT -> /servoBoard/BATT_VDD
- J3 pad 16: C_GND -> /servoBoard/BATT_VDD
- J3 pad 17: /control/EXT -> /servoBoard/BATT_VDD
- J3 pad 18: /control/EXT -> /servoBoard/BATT_VDD
- J3 pad 19: C_GND -> /servoBoard/BATT_VDD
- J3 pad 2: SPI_SCK -> /servoBoard/SPI_SCK
- J3 pad 20: C_GND -> /servoBoard/BATT_VDD
- J3 pad 3: C_GND -> /servoBoard/GND
- J3 pad 4: SPI_MISO_MOSI -> /servoBoard/SPI_MISO_MOSI
- J3 pad 5: C_GND -> /servoBoard/GND
- J3 pad 6: DOCK_1_CE -> /servoBoard/DOCK_1_CE
- J3 pad 7: DOCK_2_CE -> /servoBoard/DOCK_2_CE
- J3 pad 8: DOCK_3_CE -> /servoBoard/DOCK_3_CE
- J3 pad 9: C_GND -> /servoBoard/GND
- J4 pad 1: MOTORS_TX -> /servoBoard/GND
- J4 pad 2: MOTORS_RX -> /servoBoard/BATT_VDD
- J4 pad 3: C_GND -> /servoBoard/MOTORS_TX
- J8 pad A5: (no net) -> /control/CC1
- J8 pad B5: (no net) -> /control/CC2
- U11 pad 16: C_SW_MID -> C_SW_RIGHT
- U11 pad 17: C_SW_RIGHT -> C_SW_MID
- U11 pad 19: QC_10_N -> C_PWR_SHUTDOWN
- U11 pad 20: QC_2_P -> C_CHG_OK
- U11 pad 25: C_PWR_SHUTDOWN -> QC_10_N
- U11 pad 27: USB_TO_BUS_EN -> QC_2_P
- U11 pad 28: BATT_TO_BUS_EN -> MPU_INT
- U11 pad 42: MPU_INT -> BATT_TO_BUS_EN
- U11 pad 46: C_CHG_OK -> USB_TO_BUS_EN
- U4 pad 1: B_GND -> Net-(C18-Pad1)
- U4 pad 2: Net-(C18-Pad2) -> B_GND
- U4 pad 3: B_BATT_VDD -> Net-(R7-Pad2)
- U4 pad 4: Net-(R7-Pad2) -> Net-(R1-Pad2)
- U4 pad 5: Net-(R1-Pad2) -> B_BATT_VDD
- U4 pad 6: Net-(C18-Pad1) -> Net-(C18-Pad2)
Routing:
- net /slipRing/GND: track 0.00 -> 1414.6 mm, vias 0 -> 470
- net /slipRing/BATT_VDD: track 0.00 -> 550.2 mm, vias 0 -> 176
- net /slipRing/SPI_SCK: track 0.00 -> 236.3 mm, vias 0 -> 1
- net /slipRing/INT: track 0.00 -> 227.3 mm, vias 0 -> 72
- net /slipRing/EXT: track 0.00 -> 214.4 mm, vias 0 -> 70
- net /slipRing/SPI_MISO_MOSI: track 0.00 -> 213.8 mm, vias 0 -> 1
- net /slipRing/DOCK_1_CE: track 0.00 -> 203.2 mm, vias 0 -> 1
- net /slipRing/DOCK_2_CE: track 0.00 -> 192.3 mm, vias 0 -> 1
- net /slipRing/DOCK_3_CE: track 0.00 -> 181.2 mm, vias 0 -> 1
- net /slipRing/MOTORS_RX: track 0.00 -> 142.2 mm, vias 0 -> 1
- net C_3V3: track 0.00 -> 138.6 mm, vias 0 -> 12
- net /slipRing/MOTORS_TX: track 0.00 -> 130.4 mm, vias 0 -> 1
- net C_BATT_VDD: track 0.00 -> 125.8 mm, vias 0 -> 74
- net C_SCL: track 0.00 -> 123.7 mm, vias 0 -> 5
- net /Shoe/Shoe pads right/VCC: track 0.00 -> 120.3 mm
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- added copper zone on B.Cu, net /Shoe/Body-shoe cable.sch/BATT_VDD
- added copper zone on B.Cu, net /Shoe/Body-shoe cable.sch/EXT
- added copper zone on B.Cu, net /Shoe/Body-shoe cable.sch/GND
- added copper zone on F.Cu, net /Shoe/Body-shoe cable.sch/GND
- added copper zone on B.Cu, net /Shoe/Body-shoe cable.sch/INT
- added copper zone on B.Cu, net /Shoe/Shoe pads left/GND
- added copper zone on F.Cu, net /Shoe/Shoe pads left/GND
- added copper zone on B.Cu, net /Shoe/Shoe pads middle/GND
- added copper zone on F.Cu, net /Shoe/Shoe pads middle/GND
- added copper zone on B.Cu, net /Shoe/Shoe pads right/GND
- added copper zone on F.Cu, net /Shoe/Shoe pads right/GND
- added copper zone on B.Cu, net /battery/BAT+
- added copper zone on F.Cu, net /battery/BAT+
- added copper zone on In1.Cu, net /battery/BAT+
- added copper zone on B.Cu, net /battery/BATT_MID
- added copper zone on F.Cu, net /control/EXT
- added copper zone on B.Cu, net /debugInterface/GND
- added copper zone on B.Cu, net /power/BBV_OUTPUT
- added copper zone on B.Cu, net /power/UBV_OUTPUT
- added copper zone on B.Cu, net /servoBoard/BATT_VDD
- added copper zone on F.Cu, net /servoBoard/BATT_VDD
- added copper zone on F.Cu, net /servoBoard/EXT
- added copper zone on B.Cu, net /servoBoard/GND
- added copper zone on F.Cu, net /servoBoard/GND
- added copper zone on F.Cu, net /servoBoard/INT
- added copper zone on B.Cu, net /slipRing/BATT_VDD
- added copper zone on B.Cu, net /slipRing/EXT
- added copper zone on B.Cu, net /slipRing/GND
- added copper zone on B.Cu, net /slipRing/INT
- added copper zone on F.Cu, net B_3V3
- added copper zone on F.Cu, net B_BATT_VDD
- added copper zone on B.Cu, net B_GND
- added copper zone on F.Cu, net B_GND
- added copper zone on In1.Cu, net B_GND
- added copper zone on In2.Cu, net B_GND
- added copper zone on F.Cu, net B_INT
- added copper zone on In1.Cu, net C_3V3
- added copper zone on B.Cu, net C_BATT_VDD
- added copper zone on F.Cu, net C_BATT_VDD
- added copper zone on In2.Cu, net C_BATT_VDD
- added copper zone on B.Cu, net C_GND
- added copper zone on F.Cu, net C_GND
- added copper zone on In1.Cu, net C_GND
- added copper zone on In2.Cu, net C_GND
- added copper zone on B.Cu, net C_INT
- added copper zone on F.Cu, net C_INT
- added copper zone on F.Cu, net I_3V3
- added copper zone on B.Cu, net I_BATT_VDD
- added copper zone on F.Cu, net I_BATT_VDD
- added copper zone on F.Cu, net I_CHG_OK
- added copper zone on B.Cu, net I_GND
- added copper zone on F.Cu, net I_GND
- added copper zone on B.Cu, net I_INT
- added copper zone on F.Cu, net I_INT
- added copper zone on F.Cu, net I_PIEZO_N
- added copper zone on F.Cu, net I_SCL
- added copper zone on F.Cu, net I_START_SW
- added copper zone on F.Cu, net I_SW_MID
- added copper zone on B.Cu, net Net-(C16-Pad2)
- added copper zone on B.Cu, net Net-(C17-Pad2)
- added copper zone on F.Cu, net Net-(C18-Pad2)
- added copper zone on F.Cu, net Net-(C54-Pad1)
- added copper zone on F.Cu, net Net-(L4-Pad1)
- added copper zone on F.Cu, net Net-(Q1-Pad1)
- added copper zone on B.Cu, net USB_C_VDD
- added copper zone on F.Cu, net USB_C_VDD
Other:
- board size 193.5 x 76 mm -> 305 x 210 mm
- rule pad_to_mask_clearance: 0 -> 0.051
- rule solder_mask_min_width: 0.1 -> 0.25
- board text added: "3V3 BOOT GND"
- board text added: "3V3 GND GND GND GND"
- board text added: "BAT+"
- board text added: "BAT-"
- board text added: "BATT_VDD"
- board text added: "CLK IO GND 3V3 NC"
- board text added: "DBG"
- board text added: "ESP DBG"
- board text added: "ESP_EN ESP_TMS ESP_TCK ESP_TDI SWCLK SWDIO SWRST 3V3 GND"
- board text added: "GND EXT INT VCC"
- board text added: "GND EXT INT VDD VDD GND GND GND"
- board text added: "GND SCK GND MOSI SS4 SS5 SS6 GND VDD VDD RX TX INT EXT GND"
- board text added: "INT"
- board text added: "IO GND CLK 3V3 NC"
- board text added: "RST GND NC 3V3 NC"
- board text added: "RST NC GND 3V3 NC"
- board text added: "RoFI Body breakout v0.2 7/2021 https://ro.fi.muni.cz"
- board text added: "RoFI Shoe Center v0.2 7/2021 https://ro.fi.muni.cz"
- board text added: "RoFI Shoe Left v0.2 7/2021 https://ro.fi.muni.cz"
- board text added: "RoFI Shoe Right v0.2 7/2021 https://ro.fi.muni.cz"
- board text added: "RoFI UM Battery Board v0.2 7/2021 https://ro.fi.muni.cz"
- board text added: "RoFI UM Control Board v0.2 7/2021 https://ro.fi.muni.cz"
- board text added: "RoFI UM Display v0.2 7/2021 https://ro.fi.muni.cz"
- board text added: "SDA SCL"
- board text added: "SS3 SS2 SS1 MISO SCK"
- board text added: "ST-LINK"
- board text added: "TMS TCK TDO TDI NC"
- board text added: "TX/RX VDD GND"
- board text added: "VCC GND RST SWCLK SWDIO RX TX"
