File: hardwareModules/universalModule/hardware/controlBoard/control.sch (KiCad schematic (older format))
At the start: 36 parts, among them J1 ESP_JTAG, J4 ShoeAConnectors, J5 MOTOR_BUS, J6 MOTOR_BUS_ALT, J7 ShoeBConnectors, U6 ESP32-WROVER, U7 ICM-20948

Commit message: universalModule: Draft schematics of the new version of the control board
Parts:
- removed J1: ESP_JTAG, Connector_PinHeader_2.54mm:PinHeader_2x05_P2.54mm_Vertical, symbol Connector_Generic:Conn_02x05_Odd_Even
- removed J4: ShoeAConnectors, Connector_PinHeader_2.00mm:PinHeader_2x05_P2.00mm_Vertical, symbol Connector_Generic:Conn_02x05_Odd_Even
- removed J5: MOTOR_BUS, Connector_PinHeader_2.00mm:PinHeader_1x04_P2.00mm_Vertical, symbol Connector_Generic:Conn_01x04
- removed J6: MOTOR_BUS_ALT, Connector_PinHeader_2.00mm:PinHeader_1x03_P2.00mm_Vertical, symbol Connector_Generic:Conn_01x03
- removed J7: ShoeBConnectors, rofi:slipRingBrush, symbol Connector_Generic:Conn_01x12
- removed J?: USB_ALT, Connector_PinHeader_2.54mm:PinHeader_1x04_P2.54mm_Vertical, symbol Connector_Generic:Conn_01x04
- removed J?: BIOS_SWD, Connector_PinHeader_2.54mm:PinHeader_2x03_P2.54mm_Vertical, symbol Connector_Generic:Conn_01x05
- removed R51: 100k, Resistor_SMD:R_0402_1005Metric, symbol Device:R
- removed U7: ICM-20948, Sensor_Motion:InvenSense_QFN-24_3x3mm_P0.4mm, symbol Sensor_Motion:ICM-20948
- removed U?: STM32L432KBUx, Package_DFN_QFN:QFN-32-1EP_5x5mm_P0.5mm_EP3.45x3.45mm, symbol MCU_ST_STM32L4:STM32L432KBUx
- added C1, C25: 22u, Capacitor_SMD:C_0805_2012Metric, symbol Device:C
- added C51, C59: 470n, Capacitor_SMD:C_0402_1005Metric, symbol Device:C
- added C52, C65: 10p, Capacitor_SMD:C_0402_1005Metric, symbol Device:C
- added C60: 10u, Capacitor_SMD:C_0402_1005Metric, symbol Device:C
- added J1: DEBUG, Connector_FFC-FPC:Hirose_FH12-10S-0.5SH_1x10-1MP_P0.50mm_Horizontal, symbol Connector_Generic:Conn_01x10
- added J3: ROFICOMS, Connector_FFC-FPC:Hirose_FH12-20S-0.5SH_1x20-1MP_P0.50mm_Horizontal, symbol Connector_Generic:Conn_01x20
- added J4: MOTORS, Connector_FFC-FPC:Hirose_FH12-10S-0.5SH_1x10-1MP_P0.50mm_Horizontal, symbol Connector_Generic:Conn_01x10
- added J5: SHOE_B1, rofi:SlipRing-120220-0161, symbol Connector_Generic:Conn_01x15
- added J6: SHOE_B2, rofi:SlipRing-120220-0161, symbol Connector_Generic:Conn_01x15
- added JP1: BootSelector, Jumper:SolderJumper-3_P2.0mm_Open_TrianglePad1.0x1.5mm, symbol Jumper:SolderJumper_3_Open
- added U11: STM32F411CEUx, Package_DFN_QFN:QFN-48-1EP_7x7mm_P0.5mm_EP5.6x5.6mm, symbol MCU_ST_STM32F4:STM32F411CEUx
- added U12: HT7533-1-SOT89, Package_TO_SOT_SMD:SOT-89-3, symbol Regulator_Linear:HT75xx-1-SOT89
- added U7: MPU-6050, Sensor_Motion:InvenSense_QFN-24_4x4mm_P0.5mm, symbol Sensor_Motion:MPU-6050
- added Y1: 7D024000H01, Crystal:Crystal_SMD_2016-4Pin_2.0x1.6mm, symbol Device:Crystal_GND24
- J8: renamed from J?; symbol Connector:USB_C_Receptacle_USB2.0 -> controlBoard-rescue:USB_C_Receptacle_USB2.0-Connector
- gave numbers to parts that had none: 15
Connections:
- net BAT_VDD is gone; now on net BATT_VDD: R31.1, TP1.1
- net 3V3: now also C41.2, C42.2, J1.9 (Pin_9), JP1.3 (B), U11.1 (VBAT), U11.24 (VDD), U11.36 (VDD), U11.48 (VDD), U7.13 (VDD), U7.8 (VDDIO); no longer C41.1, C42.1
- net BATT_TO_BUS_EN: now also U11.28 (PB15)
- net BATT_VDD: now also C1.1, J3.10 (Pin_10), J3.11 (Pin_11), J4.4 (Pin_4), J4.5 (Pin_5), J4.6 (Pin_6), J5.10 (Pin_10), J5.9 (Pin_9), J6.6 (Pin_6), J6.7 (Pin_7), U12.2 (VIN)
- net BATT_VOLTAGE: now also U11.14 (PA4)
- net BIOS_RX: now also U6.29 (IO5), U11.13 (PA3); no longer U6.24 (IO2)
- net BIOS_TX: now also U6.7 (I/A/IO35), U11.12 (PA2); no longer U6.25 (IO0)
- net BUS_VOLTAGE: now also U11.10 (PA0)
- net DOCK_1_CE: now also J3.6 (Pin_6)
- net DOCK_2_CE: now also J3.7 (Pin_7)
- net DOCK_3_CE: now also J3.8 (Pin_8)
- net DOCK_4_CE: now also U6.24 (IO2), J5.5 (Pin_5); no longer U6.7 (I/A/IO35)
- net DOCK_5_CE: now also J5.6 (Pin_6)
- net DOCK_6_CE: now also J5.7 (Pin_7)
- net ESP_EN: now also U11.40 (PB4)
- net ESP_TCK: now also J1.3 (Pin_3)
- net ESP_TDI: now also J1.5 (Pin_5)
- net ESP_TDO: now also J1.4 (Pin_4)
- net ESP_TMS: now also J1.2 (Pin_2)
- net EXT: now also J3.17 (Pin_17), J3.18 (Pin_18), J5.14 (Pin_14), J6.2 (Pin_2)
- net GND: now also C41.1, C42.1, C1.2, C25.2, C51.1, C52.2, C59.2, C60.2, C65.2, J1.1 (Pin_1), J1.10 (Pin_10), J3.1 (Pin_1), J3.12 (Pin_12), J3.13 (Pin_13), J3.16 (Pin_16), J3.19 (Pin_19), J3.20 (Pin_20), J3.3 (Pin_3), J3.5 (Pin_5), J3.9 (Pin_9), J4.10 (Pin_10), J4.3 (Pin_3), J4.7 (Pin_7), J4.8 (Pin_8), J4.9 (Pin_9), J5.1 (Pin_1), J5.15 (Pin_15), J5.3 (Pin_3), J5.8 (Pin_8), J6.1 (Pin_1), J6.13 (Pin_13), J6.15 (Pin_15), J6.8 (Pin_8), JP1.1 (A), U11.23 (VSS), U11.35 (VSS), U11.47 (VSS), U11.49 (VSS), U11.8 (VSSA), U12.1 (GND), U7.1 (CLKIN), U7.11 (FSYNC), U7.18 (GND), U7.9 (AD0), Y1.2, Y1.4; no longer C41.2, C42.2
- net INT: now also J3.14 (Pin_14), J3.15 (Pin_15), J5.13 (Pin_13), J6.3 (Pin_3)
- net MOTORS_RX: now also J4.2 (Pin_2), J5.11 (Pin_11), J6.5 (Pin_5)
- net MOTORS_TX: now also J4.1 (Pin_1), J5.12 (Pin_12), J6.4 (Pin_4)
- net PWR_SHUTDOWN: now also U11.25 (PB12)
- net QC_10_N: now also U11.19 (PB1)
- net QC_10_P: now also U11.39 (PB3)
- net QC_2_M: now also U11.18 (PB0)
- net QC_2_P: now also U11.20 (PB2)
- net RXD0: now also U11.30 (PA9)
- net SPI_MISO_MOSI: now also J3.4 (Pin_4), J5.4 (Pin_4)
- net SPI_SCK: now also J3.2 (Pin_2), J5.2 (Pin_2)
- net SWCLK: now also J1.6 (Pin_6), U11.37 (PA14)
- net SWDIO: now also J1.7 (Pin_7), U11.34 (PA13)
- net SWRST: now also C59.1, J1.8 (Pin_8), U11.7 (NRST)
- net SW_LEFT: now also U11.15 (PA5)
- net SW_MID: now also U11.16 (PA6)
- net SW_RIGHT: now also U11.17 (PA7)
- net TXD0: now also U11.31 (PA10)
- net USB_C_D+: now also U11.33 (PA12)
- net USB_C_D-: now also U11.32 (PA11)
- net USB_TO_BUS_EN: now also U11.27 (PB14)
- net USB_VOLTAGE: now also U11.11 (PA1)
- net at C43.2: now also U7.10 (REGOUT)
- net BIOS_SCL renamed SCL
- net SCL: now also U11.45 (PB8), U7.23 (SCL)
- net BIOS_SDA renamed SDA
- net SDA: now also U11.43 (PB7), U7.24 (SDA)
- new net: C60.1, U11.22 (VCAP1)
- new net: JP1.2 (C), U11.44 (BOOT0)
- new net: C52.1, U11.5 (PH0), Y1.1
- new net: C65.1, U11.6 (PH1), Y1.3
- new net: C51.2, U7.20 (CPOUT)
- new net 3V3_ANALOG: C25.1, U11.9 (VDDA), U12.3 (VOUT)
- new net BUZZER_N: U11.26 (PB13)
- new net BUZZER_P: U11.29 (PA8)
- new net CHG_EN: U11.21 (PB10)
- new net CHK_OK: U11.46 (PB9)
- new net ESP_BOOT: U11.41 (PB5), U6.25 (IO0)
- new net MPU_INT: U11.42 (PB6), U7.12 (INT)
- no-connect marks 17 -> 24
Other:
- moved on the sheet: C61, C62, C63, C64, J8, R21, R22, R23, R30, R31, R32, R33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

Commit message: universalModule: Prepare electronics v0.2
Parts:
- removed C40: 470n, Capacitor_SMD:C_0402_1005Metric, symbol Device:C
- removed J3: ROFICOMS, Connector_FFC-FPC:Hirose_FH12-20S-0.5SH_1x20-1MP_P0.50mm_Horizontal, symbol Connector_Generic:Conn_01x20
- removed J4: MOTORS, Connector_FFC-FPC:Hirose_FH12-10S-0.5SH_1x10-1MP_P0.50mm_Horizontal, symbol Connector_Generic:Conn_01x10
- added J22: SHOE_OUT, rofi:Hirose_FH12-40S-0.5SH_1x40-1MP_P0.50mm_Horizontal, symbol rofi:Conn_01x40-FPC
- added R37, R38: 5k1, Resistor_SMD:R_0402_1005Metric, symbol Device:R
- C1, C25, C39, C61: LCSC (none) -> C45783
- C41, C42, C43, C51, C59, C62, C63, C64: LCSC (none) -> C47339
- J1: footprint Connector_FFC-FPC:Hirose_FH12-10S-0.5SH_1x10-1MP_P0.50mm_Horizontal -> rofi:Hirose_FH12-10S-0.5SH_1x10-1MP_P0.50mm_Horizontal; symbol Connector_Generic:Conn_01x10 -> rofi:Conn_01x10-FPC; JLCPCB_IGNORE (none) -> YES; MFR (none) -> FH12-10S-0.5SH(55); MFR_QTY (none) -> 1
- J5: JLCPCB_IGNORE (none) -> YES; MFR (none) -> 120220-0161; MFR_QTY (none) -> 15
- J6: footprint rofi:SlipRing-120220-0161 -> rofi:SlipRing-120220-0161-incomplete; symbol Connector_Generic:Conn_01x15 -> rofi:Conn_01x15_UM_slipring; JLCPCB_IGNORE (none) -> YES; MFR (none) -> 120220-0161; MFR_QTY (none) -> 8
- J8: JLCPCB_CORRECTION (none) -> 1.8;-3.3;180; LCSC (none) -> C165948
- JP1, TP1, TP3, TP4: JLCPCB_IGNORE (none) -> YES
- R21, R23: LCSC (none) -> C36871
- R22, R30, R34, R36: LCSC (none) -> C25744
- R28, R29: LCSC (none) -> C25890
- R33, R35: LCSC (none) -> C25879
- U11, U7: JLCPCB_CORRECTION (none) -> 0;0;90
- U12: JLCPCB_CORRECTION (none) -> 0;0;180
- U6: JLCPCB_CORRECTION (none) -> 0;-8.2;90; LCSC (none) -> C529591
Connections:
- net BATT_TO_BUS_EN: now also U11.42 (PB6); no longer U11.28 (PB15)
- net BATT_VDD: now also J1.MP1, J1.MP2, J22.20 (Pin_20), J22.21 (Pin_21), J22.22 (Pin_22), J22.23 (Pin_23), J22.24 (Pin_24), J22.25 (Pin_25), J22.26 (Pin_26), J22.27 (Pin_27)
- net CHK_OK: now also U11.20 (PB2); no longer U11.46 (PB9)
- net DOCK_1_CE: now also J22.35 (Pin_35)
- net DOCK_2_CE: now also J22.34 (Pin_34)
- net DOCK_3_CE: now also J22.33 (Pin_33)
- net ESP_EN: now also J1.1 (Pin_1)
- net EXT: now also J22.12 (Pin_12), J22.13 (Pin_13), J22.14 (Pin_14), J22.15 (Pin_15)
- net GND: now also J22.1 (Pin_1), J22.10 (Pin_10), J22.11 (Pin_11), J22.2 (Pin_2), J22.28 (Pin_28), J22.29 (Pin_29), J22.3 (Pin_3), J22.32 (Pin_32), J22.36 (Pin_36), J22.38 (Pin_38), J22.4 (Pin_4), J22.40 (Pin_40), J22.5 (Pin_5), J22.6 (Pin_6), J22.7 (Pin_7), J22.8 (Pin_8), J22.9 (Pin_9), J22.MP1, R37.1, R38.1; no longer J1.1 (Pin_1)
- net INT: now also J22.16 (Pin_16), J22.17 (Pin_17), J22.18 (Pin_18), J22.19 (Pin_19), J22.MP2
- net MOTORS_RX: now also J22.30 (Pin_30); no longer J6.5 (Pin_5)
- net MOTORS_TX: now also J22.31 (Pin_31); no longer J6.4 (Pin_4)
- net MPU_INT: now also U11.28 (PB15); no longer U11.42 (PB6)
- net PWR_SHUTDOWN: now also U11.19 (PB1); no longer U11.25 (PB12)
- net QC_10_N: now also U11.25 (PB12); no longer U11.19 (PB1)
- net QC_2_P: now also U11.27 (PB14); no longer U11.20 (PB2)
- net SPI_MISO_MOSI: now also J22.37 (Pin_37)
- net SPI_SCK: now also J22.39 (Pin_39)
- net SW_MID: now also U11.17 (PA7); no longer U11.16 (PA6)
- net SW_RIGHT: now also U11.16 (PA6); no longer U11.17 (PA7)
- net USB_TO_BUS_EN: now also U11.46 (PB9); no longer U11.27 (PB14)
- net CC1: now reaches J8.A5 (CC1)
- net CC1: now also R37.2
- net CC2: now reaches J8.B5 (CC2)
- net CC2: now also R38.2
- no-connect marks 24 -> 17
Other:
- note added: "Supress warning\nfrom the jumper"
- moved on the sheet: J5, R23, R30, R31, R32, TP1

Commit message: universalModule: Add final pre-production tweaks
Parts:
- J22: MFR_QTY 2 -> 1
Changed lines of the file:
@@
 F 4 "FH12-40S-0.5SH(55)" H 5100 5650 50  0001 C CNN "MFR"
 F 5 "YES" H 5100 5650 50  0001 C CNN "JLCPCB_IGNORE"
-F 6 "2" H 5100 5650 50  0001 C CNN "MFR_QTY"
+F 6 "1" H 5100 5650 50  0001 C CNN "MFR_QTY"
 	1    5100 5650
 	-1   0    0    1
